File: hardware/main_board/main_board.kicad_sch (KiCad schematic)
At the start: 33 parts, among them J1 RJ45_Shielded, J2 RJ45_Shielded, J3 Conn_01x04, J4 Conn_01x04, U1 ADS1115IDGS, U2 ADS1115IDGS, U4 TCA9548APWR

Commit message: Move ADC into sensor heads, add SSD1322 display, one I2C bus per head
Architecture:
- Each sensor head now carries the ADS1115 ADC, an MCP9808 temperature
  sensor, the EEPROM and its own LDOs. The Ethernet cable carries only
  8V, I2C and a presence-detect tie to ground.
- Drop the TCA9548A multiplexer: head 1 is on Pico I2C0 (GP0/GP1), head
  2 on I2C1 (GP2/GP3). Presence detect moves to GP4/GP5, active low.
- Replace the two I2C SSD1306 OLEDs with one 256x64 SSD1322 grayscale
  OLED on SPI1 (GP10/GP11, CS GP13, D/C GP14, RST GP15), showing both
  channels side by side.
- Main unit power: 12V input, LM317M set to 8V for the head rail, 1A 5V
  buck for the W5500-EVB-Pico, SOT-223 3.3V LDO for the OLED.

Firmware:
- New drivers: display/ssd1322.py (GS4_HMSB frame buffer), sensors/mcp9808.py
- ADS1115 continuous-conversion mode; reads never block
- PowerMeter takes two I2C buses; CalibrationManager holds one EEPROM
  driver per channel; no channel-select step anywhere
- SCPI: MEASure:TEMPerature[1|2]? returns head temperature
- Removed sensors/tca9548a.py and display/ssd1306.py

Hardware:
- Project KiCad library hardware/lib with Amphenol 132289 SMA, Amphenol
  RJHSE-5380 and Wuerth 615108150221R mid-mount RJ45 (symbols,
  footprints, 3D models), wired into both projects via RFPM_LIB
- Schematic connectors re-pointed at the new library parts
- READMEs: cable pinout, I2C topology, AD8307 front end with 3dB pad and
  1nF coupling, Hammond 1455D601BK fit analysis, power tree, schematic
  to-do lists
Parts:
- J1, J2: value RJ45_Shielded -> RJHSE-5380; footprint (none) -> rf_power_meter:RJ45_Amphenol_RJHSE5380; symbol Connector:RJ45_Shielded -> rf_power_meter:RJ45_RJHSE-5380
Changed lines of the file:
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@@
 	)
 	(symbol
-		(lib_id "Connector:RJ45_Shielded")
+		(lib_id "rf_power_meter:RJ45_RJHSE-5380")
 		(at 64.77 91.44 0)
 		(mirror x)
@@
 			)
 		)
-		(property "Value" "RJ45_Shielded"
+		(property "Value" "RJHSE-5380"
 			(at 55.88 93.9799 0)
 			(effects
@@
 			)
 		)
-		(property "Footprint" ""
+		(property "Footprint" "rf_power_meter:RJ45_Amphenol_RJHSE5380"
 			(at 64.77 92.075 90)
 			(effects
@@
 			)
 		)
-		(property "Datasheet" "~"
+		(property "Datasheet" "https://www.amphenolcanada.com/ProductSearch/drawings/AC/RJHSE538X.pdf"
 			(at 64.77 92.075 90)
 			(effects
@@
 	)
 	(symbol
-		(lib_id "Connector:RJ45_Shielded")
+		(lib_id "rf_power_meter:RJ45_RJHSE-5380")
 		(at 66.04 53.34 0)
 		(mirror x)
@@
 			)
 		)
-		(property "Value" "RJ45_Shielded"
+		(property "Value" "RJHSE-5380"
 			(at 57.15 55.8799 0)
 			(effects
@@
 			)
 		)
-		(property "Footprint" ""
+		(property "Footprint" "rf_power_meter:RJ45_Amphenol_RJHSE5380"
 			(at 66.04 53.975 90)
 			(effects
@@
 			)
 		)
-		(property "Datasheet" "~"
+		(property "Datasheet" "https://www.amphenolcanada.com/ProductSearch/drawings/AC/RJHSE538X.pdf"
 			(at 66.04 53.975 90)
 			(effects
